Commit message: chore: optimize model

File: src/track_pkg/urdf/follower.urdf.xacro (robot description, xacro)
@@ -7,4 +7,5 @@
     <xacro:property name="wheel_radius" value="0.08"/>
     <xacro:property name="wheel_width" value="0.04"/>
+    <xacro:property name="wheel_separation_length" value="0.30"/>  <!-- 前后轮距 -->
     <!-- Base link -->
     <link name="base_link">
@@ -27,4 +28,42 @@
         </inertial>
     </link>
+    <!-- Wheel Macro -->
+    <xacro:macro name="wheel" params="prefix suffix x_reflect y_reflect">
+        <link name="${prefix}_${suffix}_wheel">
+            <visual>
+                <geometry>
+                    <cylinder radius="${wheel_radius}" length="${wheel_width}"/>
+                </geometry>
+                <material name="black">
+                    <color rgba="0 0 0 1"/>
+                </material>
+            </visual>
+            <collision>
+                <geometry>
+                    <cylinder radius="${wheel_radius}" length="${wheel_width}"/>
+                </geometry>
+            </collision>
+            <inertial>
+                <mass value="0.5"/>
+                <inertia ixx="0.01" ixy="0" ixz="0" iyy="0.01" iyz="0" izz="0.01"/>
+            </inertial>
+        </link>
+        <joint name="${prefix}_${suffix}_wheel_joint" type="continuous">
+            <parent link="base_link"/>
+            <child link="${prefix}_${suffix}_wheel"/>
+            <origin xyz="${x_reflect*wheel_separation_length/2} ${y_reflect*(base_width/2 + wheel_width/2)} 0" rpy="${pi/2} 0 0"/>
+            <axis xyz="0 0 1"/>
+        </joint>
+        <gazebo reference="${prefix}_${suffix}_wheel">
+            <material>Gazebo/Black</material>
+            <mu1>1.0</mu1>
+            <mu2>1.0</mu2>
+        </gazebo>
+    </xacro:macro>
+    <!-- Create wheels -->
+    <xacro:wheel prefix="front" suffix="left"  x_reflect="1" y_reflect="1" />
+    <xacro:wheel prefix="front" suffix="right" x_reflect="1" y_reflect="-1" />
+    <xacro:wheel prefix="rear"  suffix="left"  x_reflect="-1" y_reflect="1" />
+    <xacro:wheel prefix="rear"  suffix="right" x_reflect="-1" y_reflect="-1" />
     <!-- Camera link -->
     <link name="camera_link">
@@ -44,14 +83,35 @@
         <origin xyz="${base_length/2} 0 ${base_height/2}" rpy="0 0 0"/>
     </joint>
+    <!-- Gazebo materials -->
+    <gazebo reference="base_link">
+        <material>Gazebo/Blue</material>
+        <mu1>0.2</mu1>
+        <mu2>0.2</mu2>
+    </gazebo>
     <!-- Gazebo plugin -->
     <gazebo>
         <plugin name="differential_drive_controller" filename="libgazebo_ros_diff_drive.so">
-            <leftJoint>left_wheel_joint</leftJoint>
-            <rightJoint>right_wheel_joint</rightJoint>
+            <!-- 左侧轮子 -->
+            <leftJoint>front_left_wheel_joint</leftJoint>
+            <leftJoint>rear_left_wheel_joint</leftJoint>
+            <!-- 右侧轮子 -->
+            <rightJoint>front_right_wheel_joint</rightJoint>
+            <rightJoint>rear_right_wheel_joint</rightJoint>
             <wheelSeparation>${base_width}</wheelSeparation>
             <wheelDiameter>${2*wheel_radius}</wheelDiameter>
             <robotBaseFrame>base_link</robotBaseFrame>
+            <commandTopic>cmd_vel</commandTopic>
+            <odometryTopic>odom</odometryTopic>
+            <odometryFrame>odom</odometryFrame>
+            <robotNamespace>/</robotNamespace>
             <publishWheelTF>true</publishWheelTF>
             <publishWheelJointState>true</publishWheelJointState>
+            <publishOdomTF>true</publishOdomTF>
+            <odometrySource>world</odometrySource>
+            <updateRate>50.0</updateRate>
+            <wheelAcceleration>1.0</wheelAcceleration>
+            <wheelTorque>20.0</wheelTorque>
+            <rosDebugLevel>Debug</rosDebugLevel>
+            <legacyMode>false</legacyMode>
         </plugin>
     </gazebo>

File: src/track_pkg/urdf/leader.urdf.xacro (robot description, xacro)
@@ -7,4 +7,5 @@
     <xacro:property name="wheel_radius" value="0.08"/>
     <xacro:property name="wheel_width" value="0.04"/>
+    <xacro:property name="wheel_separation_length" value="0.30"/>  <!-- 前后轮距 -->
     <!-- Base link -->
     <link name="base_link">
@@ -27,58 +28,42 @@
         </inertial>
     </link>
-    <!-- Left wheel -->
-    <link name="left_wheel">
-        <visual>
-            <geometry>
-                <cylinder radius="${wheel_radius}" length="${wheel_width}"/>
-            </geometry>
-            <material name="black">
-                <color rgba="0 0 0 1"/>
-            </material>
-        </visual>
-        <collision>
-            <geometry>
-                <cylinder radius="${wheel_radius}" length="${wheel_width}"/>
-            </geometry>
-        </collision>
-        <inertial>
-            <mass value="0.5"/>
-            <inertia ixx="0.01" ixy="0" ixz="0" iyy="0.01" iyz="0" izz="0.01"/>
-        </inertial>
-    </link>
-    <!-- Right wheel -->
-    <link name="right_wheel">
-        <visual>
-            <geometry>
-                <cylinder radius="${wheel_radius}" length="${wheel_width}"/>
-            </geometry>
-            <material name="black">
-                <color rgba="0 0 0 1"/>
-            </material>
-        </visual>
-        <collision>
-            <geometry>
-                <cylinder radius="${wheel_radius}" length="${wheel_width}"/>
-            </geometry>
-        </collision>
-        <inertial>
-            <mass value="0.5"/>
-            <inertia ixx="0.01" ixy="0" ixz="0" iyy="0.01" iyz="0" izz="0.01"/>
-        </inertial>
-    </link>
-    <!-- Left wheel joint -->
-    <joint name="left_wheel_joint" type="continuous">
-        <parent link="base_link"/>
-        <child link="left_wheel"/>
-        <origin xyz="0 ${base_width/2 + wheel_width/2} 0" rpy="${pi/2} 0 0"/>
-        <axis xyz="0 0 1"/>
-    </joint>
-    <!-- Right wheel joint -->
-    <joint name="right_wheel_joint" type="continuous">
-        <parent link="base_link"/>
-        <child link="right_wheel"/>
-        <origin xyz="0 ${-base_width/2 - wheel_width/2} 0" rpy="${pi/2} 0 0"/>
-        <axis xyz="0 0 1"/>
-    </joint>
+    <!-- Wheel Macro -->
+    <xacro:macro name="wheel" params="prefix suffix x_reflect y_reflect">
+        <link name="${prefix}_${suffix}_wheel">
+            <visual>
+                <geometry>
+                    <cylinder radius="${wheel_radius}" length="${wheel_width}"/>
+                </geometry>
+                <material name="black">
+                    <color rgba="0 0 0 1"/>
+                </material>
+            </visual>
+            <collision>
+                <geometry>
+                    <cylinder radius="${wheel_radius}" length="${wheel_width}"/>
+                </geometry>
+            </collision>
+            <inertial>
+                <mass value="0.5"/>
+                <inertia ixx="0.01" ixy="0" ixz="0" iyy="0.01" iyz="0" izz="0.01"/>
+            </inertial>
+        </link>
+        <joint name="${prefix}_${suffix}_wheel_joint" type="continuous">
+            <parent link="base_link"/>
+            <child link="${prefix}_${suffix}_wheel"/>
+            <origin xyz="${x_reflect*wheel_separation_length/2} ${y_reflect*(base_width/2 + wheel_width/2)} 0" rpy="${pi/2} 0 0"/>
+            <axis xyz="0 0 1"/>
+        </joint>
+        <gazebo reference="${prefix}_${suffix}_wheel">
+            <material>Gazebo/Black</material>
+            <mu1>1.0</mu1>
+            <mu2>1.0</mu2>
+        </gazebo>
+    </xacro:macro>
+    <!-- Create wheels -->
+    <xacro:wheel prefix="front" suffix="left"  x_reflect="1" y_reflect="1" />
+    <xacro:wheel prefix="front" suffix="right" x_reflect="1" y_reflect="-1" />
+    <xacro:wheel prefix="rear"  suffix="left"  x_reflect="-1" y_reflect="1" />
+    <xacro:wheel prefix="rear"  suffix="right" x_reflect="-1" y_reflect="-1" />
     <!-- Gazebo materials -->
     <gazebo reference="base_link">
@@ -87,19 +72,13 @@
         <mu2>0.2</mu2>
     </gazebo>
-    <gazebo reference="left_wheel">
-        <material>Gazebo/Black</material>
-        <mu1>1.0</mu1>
-        <mu2>1.0</mu2>
-    </gazebo>
-    <gazebo reference="right_wheel">
-        <material>Gazebo/Black</material>
-        <mu1>1.0</mu1>
-        <mu2>1.0</mu2>
-    </gazebo>
     <!-- Gazebo plugin -->
     <gazebo>
         <plugin name="differential_drive_controller" filename="libgazebo_ros_diff_drive.so">
-            <leftJoint>left_wheel_joint</leftJoint>
-            <rightJoint>right_wheel_joint</rightJoint>
+            <!-- 左侧轮子 -->
+            <leftJoint>front_left_wheel_joint</leftJoint>
+            <leftJoint>rear_left_wheel_joint</leftJoint>
+            <!-- 右侧轮子 -->
+            <rightJoint>front_right_wheel_joint</rightJoint>
+            <rightJoint>rear_right_wheel_joint</rightJoint>
             <wheelSeparation>${base_width}</wheelSeparation>
             <wheelDiameter>${2*wheel_radius}</wheelDiameter>

Commit message: fix: model format

File: src/track_pkg/urdf/follower.urdf.xacro (robot description, xacro)
@@ -1,3 +1,3 @@
-<?xml version="1.0" encoding="ASCII"?>
+<?xml version="1.0"?>
 <robot name="follower_robot" xmlns:xacro="http://www.ros.org/wiki/xacro">
     <!-- Property definitions -->
@@ -7,5 +7,5 @@
     <xacro:property name="wheel_radius" value="0.08"/>
     <xacro:property name="wheel_width" value="0.04"/>
-    <xacro:property name="wheel_separation_length" value="0.30"/>  <!-- 前后轮距 -->
+    <xacro:property name="wheel_separation_length" value="0.30"/>
     <!-- Base link -->
     <link name="base_link">
@@ -92,8 +92,8 @@
     <gazebo>
         <plugin name="differential_drive_controller" filename="libgazebo_ros_diff_drive.so">
-            <!-- 左侧轮子 -->
+            <!-- Left -->
             <leftJoint>front_left_wheel_joint</leftJoint>
             <leftJoint>rear_left_wheel_joint</leftJoint>
-            <!-- 右侧轮子 -->
+            <!-- Right -->
             <rightJoint>front_right_wheel_joint</rightJoint>
             <rightJoint>rear_right_wheel_joint</rightJoint>

File: src/track_pkg/urdf/leader.urdf.xacro (robot description, xacro)
@@ -1,3 +1,3 @@
-<?xml version="1.0" encoding="ASCII"?>
+<?xml version="1.0"?>
 <robot name="leader_robot" xmlns:xacro="http://www.ros.org/wiki/xacro">
     <!-- Property definitions -->
@@ -7,5 +7,5 @@
     <xacro:property name="wheel_radius" value="0.08"/>
     <xacro:property name="wheel_width" value="0.04"/>
-    <xacro:property name="wheel_separation_length" value="0.30"/>  <!-- 前后轮距 -->
+    <xacro:property name="wheel_separation_length" value="0.30"/>
     <!-- Base link -->
     <link name="base_link">
@@ -75,8 +75,8 @@
     <gazebo>
         <plugin name="differential_drive_controller" filename="libgazebo_ros_diff_drive.so">
-            <!-- 左侧轮子 -->
+            <!-- Left -->
             <leftJoint>front_left_wheel_joint</leftJoint>
             <leftJoint>rear_left_wheel_joint</leftJoint>
-            <!-- 右侧轮子 -->
+            <!-- Right -->
             <rightJoint>front_right_wheel_joint</rightJoint>
             <rightJoint>rear_right_wheel_joint</rightJoint>

Commit message: chore: add camera height

File: src/track_pkg/urdf/follower.urdf.xacro (robot description, xacro)
@@ -81,5 +81,5 @@
         <parent link="base_link"/>
         <child link="camera_link"/>
-        <origin xyz="${base_length/2} 0 ${base_height/2}" rpy="0 0 0"/>
+        <origin xyz="${base_length/2} 0 ${base_height + 0.1}" rpy="-0.1 0 0"/>
     </joint>
     <!-- Gazebo materials -->

Commit message: chore: add more logs

File: src/track_pkg/urdf/follower.urdf.xacro (robot description, xacro)
@@ -81,5 +81,5 @@
         <parent link="base_link"/>
         <child link="camera_link"/>
-        <origin xyz="${base_length/2} 0 ${base_height + 0.1}" rpy="-0.1 0 0"/>
+        <origin xyz="${base_length/2} 0 ${base_height + 0.1}" rpy="0 0 0"/>
     </joint>
     <!-- Gazebo materials -->
