Commit message: fix: model config and cmakelist

File: src/track_pkg/urdf/leader.urdf.xacro (robot description, xacro)
@@ -27,4 +27,74 @@
         </inertial>
     </link>
+    <!-- Left wheel -->
+    <link name="left_wheel">
+        <visual>
+            <geometry>
+                <cylinder radius="${wheel_radius}" length="${wheel_width}"/>
+            </geometry>
+            <material name="black">
+                <color rgba="0 0 0 1"/>
+            </material>
+        </visual>
+        <collision>
+            <geometry>
+                <cylinder radius="${wheel_radius}" length="${wheel_width}"/>
+            </geometry>
+        </collision>
+        <inertial>
+            <mass value="0.5"/>
+            <inertia ixx="0.01" ixy="0" ixz="0" iyy="0.01" iyz="0" izz="0.01"/>
+        </inertial>
+    </link>
+    <!-- Right wheel -->
+    <link name="right_wheel">
+        <visual>
+            <geometry>
+                <cylinder radius="${wheel_radius}" length="${wheel_width}"/>
+            </geometry>
+            <material name="black">
+                <color rgba="0 0 0 1"/>
+            </material>
+        </visual>
+        <collision>
+            <geometry>
+                <cylinder radius="${wheel_radius}" length="${wheel_width}"/>
+            </geometry>
+        </collision>
+        <inertial>
+            <mass value="0.5"/>
+            <inertia ixx="0.01" ixy="0" ixz="0" iyy="0.01" iyz="0" izz="0.01"/>
+        </inertial>
+    </link>
+    <!-- Left wheel joint -->
+    <joint name="left_wheel_joint" type="continuous">
+        <parent link="base_link"/>
+        <child link="left_wheel"/>
+        <origin xyz="0 ${base_width/2 + wheel_width/2} 0" rpy="${pi/2} 0 0"/>
+        <axis xyz="0 0 1"/>
+    </joint>
+    <!-- Right wheel joint -->
+    <joint name="right_wheel_joint" type="continuous">
+        <parent link="base_link"/>
+        <child link="right_wheel"/>
+        <origin xyz="0 ${-base_width/2 - wheel_width/2} 0" rpy="${pi/2} 0 0"/>
+        <axis xyz="0 0 1"/>
+    </joint>
+    <!-- Gazebo materials -->
+    <gazebo reference="base_link">
+        <material>Gazebo/Red</material>
+        <mu1>0.2</mu1>
+        <mu2>0.2</mu2>
+    </gazebo>
+    <gazebo reference="left_wheel">
+        <material>Gazebo/Black</material>
+        <mu1>1.0</mu1>
+        <mu2>1.0</mu2>
+    </gazebo>
+    <gazebo reference="right_wheel">
+        <material>Gazebo/Black</material>
+        <mu1>1.0</mu1>
+        <mu2>1.0</mu2>
+    </gazebo>
     <!-- Gazebo plugin -->
     <gazebo>
@@ -40,4 +110,10 @@
             <odometryTopic>leader/odom</odometryTopic>
             <odometryFrame>leader/odom</odometryFrame>
+            <updateRate>50</updateRate>
+            <wheelAcceleration>1.0</wheelAcceleration>
+            <wheelTorque>20</wheelTorque>
+            <rosDebugLevel>Debug</rosDebugLevel>
+            <publishOdomTF>true</publishOdomTF>
+            <odometrySource>world</odometrySource>
         </plugin>
     </gazebo>

Commit message: fix: img_view window

File: src/track_pkg/urdf/leader.urdf.xacro (robot description, xacro)
@@ -24,6 +24,6 @@
         </collision>
         <inertial>
-            <mass value="5.0"/>
-            <inertia ixx="0.1" ixy="0" ixz="0" iyy="0.1" iyz="0" izz="0.1"/>
+            <mass value="1.0"/>
+            <inertia ixx="0.01" ixy="0" ixz="0" iyy="0.01" iyz="0" izz="0.01"/>
         </inertial>
     </link>
@@ -45,6 +45,6 @@
             </collision>
             <inertial>
-                <mass value="0.5"/>
-                <inertia ixx="0.01" ixy="0" ixz="0" iyy="0.01" iyz="0" izz="0.01"/>
+                <mass value="0.1"/>
+                <inertia ixx="0.001" ixy="0" ixz="0" iyy="0.001" iyz="0" izz="0.001"/>
             </inertial>
         </link>

Commit message: try fix: track lost

File: src/track_pkg/urdf/leader.urdf.xacro (robot description, xacro)
@@ -8,4 +8,7 @@
     <xacro:property name="wheel_width" value="0.04"/>
     <xacro:property name="wheel_separation_length" value="0.30"/>
+    <xacro:property name="marker_width" value="0.2"/>
+    <xacro:property name="marker_height" value="0.2"/>
+    <xacro:property name="marker_thickness" value="0.01"/>
     <!-- Base link -->
     <link name="base_link">
@@ -14,6 +17,6 @@
                 <box size="${base_length} ${base_width} ${base_height}"/>
             </geometry>
-            <material name="red">
-                <color rgba="1 0 0 1"/>
+            <material name="bright_blue">
+                <color rgba="0 0.5 1 1"/>
             </material>
         </visual>
@@ -28,4 +31,51 @@
         </inertial>
     </link>
+    <!-- 添加后部标记板 -->
+    <link name="marker_board">
+        <visual>
+            <geometry>
+                <box size="${marker_thickness} ${marker_width} ${marker_height}"/>
+            </geometry>
+            <material name="checker_pattern">
+                <color rgba="1 1 0 1"/>  <!-- 黄色，更容易被识别 -->
+            </material>
+        </visual>
+        <collision>
+            <geometry>
+                <box size="${marker_thickness} ${marker_width} ${marker_height}"/>
+            </geometry>
+        </collision>
+        <inertial>
+            <mass value="0.1"/>
+            <inertia ixx="0.001" ixy="0" ixz="0" iyy="0.001" iyz="0" izz="0.001"/>
+        </inertial>
+    </link>
+    <!-- 标记板关节 -->
+    <joint name="marker_board_joint" type="fixed">
+        <parent link="base_link"/>
+        <child link="marker_board"/>
+        <origin xyz="${-base_length/2 - marker_thickness/2} 0 ${base_height/2}" rpy="0 0 0"/>
+    </joint>
+    <!-- 添加顶部标记图案 -->
+    <link name="top_pattern">
+        <visual>
+            <geometry>
+                <box size="${marker_width} ${marker_width} ${marker_thickness}"/>
+            </geometry>
+            <material name="pattern">
+                <color rgba="1 0.8 0 1"/>  <!-- 金黄色 -->
+            </material>
+        </visual>
+        <inertial>
+            <mass value="0.01"/>
+            <inertia ixx="0.001" ixy="0" ixz="0" iyy="0.001" iyz="0" izz="0.001"/>
+        </inertial>
+    </link>
+    <!-- 顶部图案关节 -->
+    <joint name="top_pattern_joint" type="fixed">
+        <parent link="base_link"/>
+        <child link="top_pattern"/>
+        <origin xyz="0 0 ${base_height/2 + marker_thickness/2}" rpy="0 0 0"/>
+    </joint>
     <!-- Wheel Macro -->
     <xacro:macro name="wheel" params="prefix suffix x_reflect y_reflect">
@@ -70,7 +120,14 @@
     <!-- Gazebo materials -->
     <gazebo reference="base_link">
-        <material>Gazebo/Red</material>
+        <material>Gazebo/Blue</material>
         <mu1>0.2</mu1>
         <mu2>0.2</mu2>
+    </gazebo>
+    <!-- 为新添加的部件设置Gazebo材质 -->
+    <gazebo reference="marker_board">
+        <material>Gazebo/Yellow</material>
+    </gazebo>
+    <gazebo reference="top_pattern">
+        <material>Gazebo/Yellow</material>
     </gazebo>
     <!-- Gazebo plugin -->

Commit message: fix: model material

File: src/track_pkg/urdf/leader.urdf.xacro (robot description, xacro)
@@ -17,7 +17,5 @@
                 <box size="${base_length} ${base_width} ${base_height}"/>
             </geometry>
-            <material name="bright_blue">
-                <color rgba="0 0.5 1 1"/>
-            </material>
+            <material name="Gazebo/Blue"/>
         </visual>
         <collision>
@@ -37,7 +35,5 @@
                 <box size="${marker_thickness} ${marker_width} ${marker_height}"/>
             </geometry>
-            <material name="checker_pattern">
-                <color rgba="1 1 0 1"/>  <!-- 黄色，更容易被识别 -->
-            </material>
+            <material name="Gazebo/Yellow"/>
         </visual>
         <collision>
@@ -63,7 +59,5 @@
                 <box size="${marker_width} ${marker_width} ${marker_thickness}"/>
             </geometry>
-            <material name="pattern">
-                <color rgba="1 0.8 0 1"/>  <!-- 金黄色 -->
-            </material>
+            <material name="Gazebo/Yellow"/>
         </visual>
         <inertial>
@@ -85,7 +79,5 @@
                     <cylinder radius="${wheel_radius}" length="${wheel_width}"/>
                 </geometry>
-                <material name="black">
-                    <color rgba="0 0 0 1"/>
-                </material>
+                <material name="Gazebo/Black"/>
             </visual>
             <collision>
